File: rover_bms_ble_controller_hw/MCU&LEDS.kicad_sch (KiCad schematic)
At the start: 57 parts, among them T2 BC817-40(SOT23), T3 BC817-40(SOT23), U2 SY8089AAAC(SOT23-5), U3 ESP32-S3-WROOM-1-N8R8, U4 CH340X(MSOP-10)

Commit message: Update
Parts:
- removed D3: 1N5819S4/SOD123, OLIMEX_Diodes-FP:SOD-123_1C-2A_KA, symbol ESP32-S3-DevKit-LiPo_Rev_B:D_Schottky
- removed R10, R13: 1k/R0402, OLIMEX_RLC-FP:R_0402_5MIL_DWS, symbol ESP32-S3-DevKit-LiPo_Rev_B:R
- removed R11: 5.1k/R0603, OLIMEX_RLC-FP:R_0603_5MIL_DWS, symbol ESP32-S3-DevKit-LiPo_Rev_B:R
- removed R14, R17: 2.2k/R0402, OLIMEX_RLC-FP:R_0402_5MIL_DWS, symbol ESP32-S3-DevKit-LiPo_Rev_B:R
- removed R16: NA/R0402, OLIMEX_RLC-FP:R_0402_5MIL_DWS, symbol ESP32-S3-DevKit-LiPo_Rev_B:R
- removed R18: 10k/R0402, OLIMEX_RLC-FP:R_0402_5MIL_DWS, symbol ESP32-S3-DevKit-LiPo_Rev_B:R
- removed R8: 100R/R0402, OLIMEX_RLC-FP:R_0402_5MIL_DWS, symbol ESP32-S3-DevKit-LiPo_Rev_B:R
- removed R9: 4.7k/R0402, OLIMEX_RLC-FP:R_0402_5MIL_DWS, symbol ESP32-S3-DevKit-LiPo_Rev_B:R
- removed T2, T3: BC817-40(SOT23), OLIMEX_Transistors-FP:SOT23, symbol ESP32-S3-DevKit-LiPo_Rev_B:Q_NPN_BEC
- removed U4: CH340X(MSOP-10), OLIMEX_IC-FP:MSOP-10_Pitch-0.5mm_3.00x3.00x1.00mm, symbol ESP32-S3-DevKit-LiPo_Rev_B:CH340E(MSOP-10)
- removed USB-UART2: USB-C-16P-F(A40-00119-A52-12), OLIMEX_Connectors-FP:USB2.0_TYPE-C(A40-00119-A52-12), symbol ESP32-S3-DevKit-LiPo_Rev_B:USB2.0_TYPE-C(A40-00119-A52-12)
- removed pUEXT2: BM10B-SRSS-TB, OLIMEX_Connectors-FP:BM10B-SRSS-TB, symbol ESP32-S3-DevKit-LiPo_Rev_B:CONN_01X10
- added C10, C9: 47uF/50V, Capacitor_SMD:CP_Elec_6.3x7.7, symbol ESP32-S3-DevKit-LiPo_Rev_B:C
- added C11, C5, C7, C_BOOT2: 100nF/50V, OLIMEX_RLC-FP:C_0603_5MIL_DWS, symbol ESP32-S3-DevKit-LiPo_Rev_B:C
- added C12: 33pF/50V, OLIMEX_RLC-FP:C_0603_5MIL_DWS, symbol ESP32-S3-DevKit-LiPo_Rev_B:C
- added C18, C21: 22uF/6.3V/20%/X5R/C0603, OLIMEX_RLC-FP:C_0603_5MIL_DWS, symbol ESP32-S3-DevKit-LiPo_Rev_B:C
- added C19, C20: 100nF/10V/10%/X7R/C0402, OLIMEX_RLC-FP:C_0402_5MIL_DWS, symbol ESP32-S3-DevKit-LiPo_Rev_B:C
- added C2: 100uF/50V, Capacitor_SMD:CP_Elec_8x10.5, symbol ESP32-S3-DevKit-LiPo_Rev_B:C
- added C3, C4: 4.7uF/50V, Capacitor_SMD:CP_Elec_4x5.7, symbol ESP32-S3-DevKit-LiPo_Rev_B:C
- added C8: 1nF/50V, OLIMEX_RLC-FP:C_0603_5MIL_DWS, symbol ESP32-S3-DevKit-LiPo_Rev_B:C
- added IC2: TXS0108E, TXS0108E:PW_R-PDSO-G20, symbol TXS0108E:TXS0108E
- added L2: 4.7uH, Inductor_SMD:L_Sunlord_MWSA1003S, symbol ESP32-S3-DevKit-LiPo_Rev_B:L
- added R3: 100k/R0603, OLIMEX_RLC-FP:R_0603_5MIL_DWS, symbol ESP32-S3-DevKit-LiPo_Rev_B:R
- added R4: 1k/R0603, OLIMEX_RLC-FP:R_0603_5MIL_DWS, symbol ESP32-S3-DevKit-LiPo_Rev_B:R
- added R5: 31.6k/R0603, OLIMEX_RLC-FP:R_0603_5MIL_DWS, symbol ESP32-S3-DevKit-LiPo_Rev_B:R
- added R6: 19.1k/R0603, OLIMEX_RLC-FP:R_0603_5MIL_DWS, symbol ESP32-S3-DevKit-LiPo_Rev_B:R
- added U2: LMR51450SDRRR, Libs:CONV_LMR51450SDRRR, symbol LMR51450SDRRR:LMR51450SDRRR
- C6: value 100nF/10V/10%/X7R/C0402 -> 1nF/50V; footprint OLIMEX_RLC-FP:C_0402_5MIL_DWS -> OLIMEX_RLC-FP:C_0603_5MIL_DWS; Fieldname 1 Value 1 -> (none); JLCPCB (none) -> C5534307
- R12: value 5.1k/R0603 -> 100k/R0603
- renumbered C2 to C13, C3 to C14, C4 to C15, C5 to C16, C7 to C17, D11 to D10, D12 to D11, D13 to D12, D14 to D13, D4 to D3, D5 to D4, D6 to D5, D7 to D6, D8 to D7, D9 to D8, D10 to D9, L2 to L3, R6 to R10, R7 to R11, R15 to R13, R19 to R14, R20 to R15, R21 to R16, R22 to R17, R23 to R18, R3 to R2, R2 to R7, R5 to R8, R4 to R9, U2 to U3, U3 to U4
Connections:
- net +3.3V: now also R12.2, C18.1, C19.2, IC2.10 (OE), IC2.2 (VCCA); no longer C6.1
- net +5V: now also C10.1, C11.2, C20.2, C21.1, C7.2, C8.2, C9.1, IC2.19 (VCCB), L2.2, R3.2, R4.2
- net GND: now also C6.1, C10.2, C11.1, C18.2, C19.1, C2.2, C20.1, C21.2, C3.2, C4.2, C5.1, C7.1, C8.1, C9.2, IC2.11 (GND), R5.1, R6.1, U2.13 (PGND), U2.8 (AGND); no longer C6.2
- net GPIO11\FSPID(SPI3_MOSI): now also IC2.1 (A1); no longer D4.1 (DI), LED_DI/CI2.1
- net GPIO12\FSPICLK(SPI3_CLK): now also IC2.3 (A2); no longer D4.2 (CI), LED_DI/CI2.2
- new net: C_BOOT2.1, L2.1, U2.1 (SW), U2.2 (SW), U2.3 (SW)
- new net: C_BOOT2.2, U2.4 (BOOT)
- new net: R5.2, U2.6 (RT)
- new net: C12.1, R3.1, R6.2, U2.7 (FB)
- new net: C12.2, R4.1
- new net +24V: C2.1, C3.1, C4.1, C5.2, C6.2, U2.10 (VIN), U2.11 (VIN), U2.12 (VIN), U2.9 (EN)
- new net LED_SPI_CLK: D4.2 (CI), IC2.18 (B2), LED_DI/CI2.2
- new net LED_SPI_MOSI: D4.1 (DI), IC2.20 (B1), LED_DI/CI2.1
- no-connect marks 4 -> 15
Other:
- note added: "Level Shifter"
- note removed: "0"
- note removed: "1"
- note removed: "Auto program"
- note removed: "DTR RTS->EN IO0"
- note removed: "USB to UART"
- note removed: "pUEXT"
- moved on the sheet: C15, C16, D2, L3, R10, R7, R8, R9, U3

Commit message: Final version
Parts:
- removed C11, C7, C_BOOT2: 100nF/50V, OLIMEX_RLC-FP:C_0603_5MIL_DWS, symbol ESP32-S3-DevKit-LiPo_Rev_B:C
- removed C16: 22uF/6.3V/20%/X5R/C0603, OLIMEX_RLC-FP:C_0603_5MIL_DWS, symbol ESP32-S3-DevKit-LiPo_Rev_B:C
- removed C19: 100nF/10V/10%/X7R/C0402, OLIMEX_RLC-FP:C_0402_5MIL_DWS, symbol ESP32-S3-DevKit-LiPo_Rev_B:C
- removed D3: 1N5819S4/SOD123, OLIMEX_Diodes-FP:SOD-123_1C-2A_KA, symbol ESP32-S3-DevKit-LiPo_Rev_B:D_Schottky
- removed IC2: TXS0108E, TXS0108E:PW_R-PDSO-G20, symbol TXS0108E:TXS0108E
- removed LED2: LED/Green/0603, OLIMEX_LEDs-FP:LED_0603_KA, symbol ESP32-S3-DevKit-LiPo_Rev_B:LED
- removed LED_DI/CI2, LED_DI/CI3, LED_DO/CO2, LED_DO/CO3: DW02S, OLIMEX_Connectors-FP:LIPO_BAT_VERTICAL_DW02S, symbol ESP32-S3-DevKit-LiPo_Rev_B:BAT_CON
- removed R13: 2.2k/R0402, OLIMEX_RLC-FP:R_0402_5MIL_DWS, symbol ESP32-S3-DevKit-LiPo_Rev_B:R
- removed R16: 100R/R0402, OLIMEX_RLC-FP:R_0402_5MIL_DWS, symbol ESP32-S3-DevKit-LiPo_Rev_B:R
- removed R17, R18: 0k/R0603, OLIMEX_RLC-FP:R_0603_5MIL_DWS, symbol ESP32-S3-DevKit-LiPo_Rev_B:R
- removed R2: 10k/R0402, OLIMEX_RLC-FP:R_0402_5MIL_DWS, symbol ESP32-S3-DevKit-LiPo_Rev_B:R
- removed U2: LMR51450SDRRR, Libs:CONV_LMR51450SDRRR, symbol LMR51450SDRRR:LMR51450SDRRR
- removed USB-OTG2: USB-C-16P-F(A40-00119-A52-12), OLIMEX_Connectors-FP:USB2.0_TYPE-C(A40-00119-A52-12), symbol ESP32-S3-DevKit-LiPo_Rev_B:USB2.0_TYPE-C(A40-00119-A52-12)
- added C12, C2, C22: 100nF/50V/0603, Capacitor_SMD:C_0603_1608Metric, symbol ESP32-S3-DevKit-LiPo_Rev_B:C
- added C17: 47uF/50V, Capacitor_SMD:CP_Elec_6.3x7.7, symbol ESP32-S3-DevKit-LiPo_Rev_B:C
- added C9: 1nF/50V/0603, Capacitor_SMD:C_0603_1608Metric, symbol ESP32-S3-DevKit-LiPo_Rev_B:C
- added IC2: TXS0108E, MechatronicsAcademy:PW_R-PDSO-G20, symbol MechatronicsAcademy:TXS0108E
- added J10: DO_OUT, MechatronicsAcademy:TestPoint_Pad, symbol MechatronicsAcademy:Conn_01x01_Pin
- added J11: CO_OUT, MechatronicsAcademy:TestPoint_Pad, symbol MechatronicsAcademy:Conn_01x01_Pin
- added J12: DO_IN, MechatronicsAcademy:TestPoint_Pad, symbol MechatronicsAcademy:Conn_01x01_Pin
- added J13: CI_IN, MechatronicsAcademy:TestPoint_Pad, symbol MechatronicsAcademy:Conn_01x01_Pin
- added J14: DO_OUT_2, MechatronicsAcademy:TestPoint_Pad, symbol MechatronicsAcademy:Conn_01x01_Pin
- added J15: DI_IN_2, MechatronicsAcademy:TestPoint_Pad, symbol MechatronicsAcademy:Conn_01x01_Pin
- added J16: CO_OUT_2, MechatronicsAcademy:TestPoint_Pad, symbol MechatronicsAcademy:Conn_01x01_Pin
- added J17: CI_IN_2, MechatronicsAcademy:TestPoint_Pad, symbol MechatronicsAcademy:Conn_01x01_Pin
- added J2: +24V_PAD, MechatronicsAcademy:TestPoint_Pad_1, symbol MechatronicsAcademy:Conn_01x01_Pin
- added J3: IN_+5, MechatronicsAcademy:TestPoint_Pad_1, symbol MechatronicsAcademy:Conn_01x01_Pin
- added J4: OUT_+5, MechatronicsAcademy:TestPoint_Pad_1, symbol MechatronicsAcademy:Conn_01x01_Pin
- added J5, J8: GND_IN, MechatronicsAcademy:TestPoint_Pad_1, symbol MechatronicsAcademy:Conn_01x01_Pin
- added J6, J9: GND_OUT, MechatronicsAcademy:TestPoint_Pad_1, symbol MechatronicsAcademy:Conn_01x01_Pin
- added J7: GND_PAD, MechatronicsAcademy:TestPoint_Pad_1, symbol MechatronicsAcademy:Conn_01x01_Pin
- added R15: 100/R0603, Resistor_SMD:R_0603_1608Metric_Pad0.98x0.95mm_HandSolder, symbol ESP32-S3-DevKit-LiPo_Rev_B:R
- added R5: 10k/R0603, Resistor_SMD:R_0603_1608Metric_Pad0.98x0.95mm_HandSolder, symbol ESP32-S3-DevKit-LiPo_Rev_B:R
- added U2: LMR51450SDRRR, MechatronicsAcademy:LMR51450SDRRR, symbol MechatronicsAcademy:LMR51450SDRRR
- added USB-C2: USB2.0_TYPE-C(A40-00119-A52-12), MechatronicsAcademy:USB2.0_TYPE-C-ONLY-PADS, symbol MechatronicsAcademy:USB2.0_TYPE-C(A40-00119-A52-12)
- BUT2, RST2: JLCPCB (none) -> C2910672
- C10: renamed from C9; JLCPCB (none) -> C2163587; JLPCB C2163587 -> (none)
- C11: renamed from C10; JLCPCB (none) -> C2163587; JLPCB C2163587 -> (none)
- C13: renamed from C12; value 33pF/50V -> 33pF/50V/0603; footprint OLIMEX_RLC-FP:C_0603_5MIL_DWS -> Capacitor_SMD:C_0603_1608Metric; JLCPCB C2180469 -> C77035
- C14: renamed from C13; value 22uF/6.3V/20%/X5R/C0603 -> 22uF/10V/X5R/0603; footprint OLIMEX_RLC-FP:C_0603_5MIL_DWS -> Capacitor_SMD:C_0603_1608Metric; JLCPCB (none) -> C84419
- C15: renamed from C14; value 100nF/10V/10%/X7R/C0402 -> 100nF/50V/0603; footprint OLIMEX_RLC-FP:C_0402_5MIL_DWS -> Capacitor_SMD:C_0603_1608Metric; JLCPCB (none) -> C77055
- C16: renamed from C15; value 22uF/6.3V/20%/X5R/C0603 -> 22uF/10V/X5R/0603; footprint OLIMEX_RLC-FP:C_0603_5MIL_DWS -> Capacitor_SMD:C_0603_1608Metric; JLCPCB (none) -> C84419
- C18: renamed from C17; value 1uF/10V/10%/X5R/C0603 -> 1uF/10V/X5R/0603; footprint OLIMEX_RLC-FP:C_0603_5MIL_DWS -> Capacitor_SMD:C_0603_1608Metric; JLCPCB (none) -> C3862113
- C19: renamed from C20; value 100nF/10V/10%/X7R/C0402 -> 100nF/50V/0603; footprint OLIMEX_RLC-FP:C_0402_5MIL_DWS -> Capacitor_SMD:C_0603_1608Metric; JLCPCB (none) -> C77055
- C20: renamed from C21; value 22uF/6.3V/20%/X5R/C0603 -> 22uF/10V/X5R/0603; footprint OLIMEX_RLC-FP:C_0603_5MIL_DWS -> Capacitor_SMD:C_0603_1608Metric; JLCPCB (none) -> C84419
- C21: renamed from C18; value 22uF/6.3V/20%/X5R/C0603 -> 22uF/10V/X5R/0603; footprint OLIMEX_RLC-FP:C_0603_5MIL_DWS -> Capacitor_SMD:C_0603_1608Metric; JLCPCB (none) -> C84419
- C6: renamed from C5; value 100nF/50V -> 100nF/50V/0603; footprint OLIMEX_RLC-FP:C_0603_5MIL_DWS -> Capacitor_SMD:C_0603_1608Metric; JLCPCB C6715111 -> C77055
- C7: renamed from C6; value 1nF/50V -> 1nF/50V/0603; footprint OLIMEX_RLC-FP:C_0603_5MIL_DWS -> Capacitor_SMD:C_0603_1608Metric; JLCPCB C5534307 -> C71653
- C8: value 1nF/50V -> 100nF/50V/0603; footprint OLIMEX_RLC-FP:C_0603_5MIL_DWS -> Capacitor_SMD:C_0603_1608Metric; JLCPCB C5534307 -> C77055
- D10: renamed from D11; value APA102 -> SK9822; JLCPCB (none) -> C2829089
- D11: renamed from D12; value APA102 -> SK9822; JLCPCB (none) -> C2829089
- D12: renamed from D13; value APA102 -> SK9822; JLCPCB (none) -> C2829089
- D2: Fieldname 1 Value 1 -> (none); Fieldname2 Value2 -> (none); Fieldname3 Value3 -> (none); JLCPCB (none) -> C2939006
- D3: renamed from D4; value APA102 -> SK9822; JLCPCB (none) -> C2829089
- D4: renamed from D5; value APA102 -> SK9822; JLCPCB (none) -> C2829089
- D5: renamed from D6; value APA102 -> SK9822; JLCPCB (none) -> C2829089
- D6: renamed from D7; value APA102 -> SK9822; JLCPCB (none) -> C2829089
- D7: renamed from D8; value APA102 -> SK9822; JLCPCB (none) -> C2829089
- D8: renamed from D9; value APA102 -> SK9822; JLCPCB (none) -> C2829089
- D9: renamed from D10; value APA102 -> SK9822; JLCPCB (none) -> C2829089
- L3: JLCPCB (none) -> C6364793
- R10: value 49.9k/1%/R0402 -> 49.9k/1%/R0603; footprint OLIMEX_RLC-FP:R_0402_5MIL_DWS -> Resistor_SMD:R_0603_1608Metric_Pad0.98x0.95mm_HandSolder; JLCPCB (none) -> C23184
- R11: value 10k/R0402 -> 10k/R0603; footprint OLIMEX_RLC-FP:R_0402_5MIL_DWS -> Resistor_SMD:R_0603_1608Metric_Pad0.98x0.95mm_HandSolder; Fieldname 1 Value 1 -> (none); Fieldname2 Value2 -> (none); Fieldname3 Value3 -> (none); JLCPCB (none) -> C95204
- R12: footprint OLIMEX_RLC-FP:R_0603_5MIL_DWS -> Resistor_SMD:R_0603_1608Metric_Pad0.98x0.95mm_HandSolder; JLCPCB (none) -> C100048
- R13: renamed from R14; footprint OLIMEX_RLC-FP:R_0603_5MIL_DWS -> Resistor_SMD:R_0603_1608Metric_Pad0.98x0.95mm_HandSolder; JLCPCB (none) -> C14677
- R14: renamed from R15; footprint OLIMEX_RLC-FP:R_0603_5MIL_DWS -> Resistor_SMD:R_0603_1608Metric_Pad0.98x0.95mm_HandSolder; JLCPCB (none) -> C14677
- R2: renamed from R3; footprint OLIMEX_RLC-FP:R_0603_5MIL_DWS -> Resistor_SMD:R_0603_1608Metric_Pad0.98x0.95mm_HandSolder; JLCPCB (none) -> C100048
- R3: renamed from R4; footprint OLIMEX_RLC-FP:R_0603_5MIL_DWS -> Resistor_SMD:R_0603_1608Metric_Pad0.98x0.95mm_HandSolder; JLCPCB (none) -> C110776
- R4: renamed from R5; footprint OLIMEX_RLC-FP:R_0603_5MIL_DWS -> Resistor_SMD:R_0603_1608Metric_Pad0.98x0.95mm_HandSolder; JLCPCB (none) -> C861351
- R6: footprint OLIMEX_RLC-FP:R_0603_5MIL_DWS -> Resistor_SMD:R_0603_1608Metric_Pad0.98x0.95mm_HandSolder; JLCPCB (none) -> C173754
- R7: value 220k/R0402 -> 2200k/R0603; footprint OLIMEX_RLC-FP:R_0402_5MIL_DWS -> Resistor_SMD:R_0603_1608Metric_Pad0.98x0.95mm_HandSolder; Fieldname 1 Value 1 -> (none); Fieldname2 Value2 -> (none); Fieldname3 Value3 -> (none); JLCPCB (none) -> C123420
- R8: value 220k/R0402 -> 220k/R0603; footprint OLIMEX_RLC-FP:R_0402_5MIL_DWS -> Resistor_SMD:R_0603_1608Metric_Pad0.98x0.95mm_HandSolder; JLCPCB (none) -> C123420
- R9: value 470k/R0402 -> 470k/R0603; footprint OLIMEX_RLC-FP:R_0402_5MIL_DWS -> Resistor_SMD:R_0603_1608Metric_Pad0.98x0.95mm_HandSolder; Fieldname 1 Value 1 -> (none); Fieldname2 Value2 -> (none); Fieldname3 Value3 -> (none); JLCPCB (none) -> C114622
- U3: JLCPCB (none) -> C78988
- U4: JLCPCB (none) -> C2913201
- renumbered C2 to C3, C3 to C4, C4 to C5
Connections:
- net +24V: now also J2.1 (Pin_1), U2.10 (VIN), U2.11 (VIN), U2.12 (VIN), U2.9 (EN)
- net +3.3V: now also C17.1, C22.2, IC2.10 (OE), IC2.2 (VCCA), R5.2
- net +5V: now also C16.1, D2.1 (K), R7.2, U3.1 (EN), U3.4 (IN), C12.2, C9.2, IC2.19 (VCCB), J3.1 (Pin_1), J4.1 (Pin_1); no longer D2.2 (A), R7.1
- net GND: now also R9.1, C12.1, C17.2, C22.1, C9.1, IC2.11 (GND), J5.1 (Pin_1), J6.1 (Pin_1), J7.1 (Pin_1), J8.1 (Pin_1), J9.1 (Pin_1), U2.13 (PGND), U2.8 (AGND), USB-C2.A1 (GND), USB-C2.A12 (GND), USB-C2.B1 (GND), USB-C2.B12 (GND); no longer R9.2
- net GPIO0\BUT1: now also R15.2
- net GPIO11\FSPID(SPI3_MOSI): now also IC2.3 (A2)
- net GPIO12\FSPICLK(SPI3_CLK): now also IC2.1 (A1)
- net GPIO19\USB_D-: now also USB-C2.A7 (DN1), USB-C2.B7 (DN2)
- net GPIO20\USB_D+: now also USB-C2.A6 (DP1), USB-C2.B6 (DP2)
- net GPIO5\PWR_SENS: now also R7.1, R9.2; no longer R7.2, R9.1
- net LED_SPI_CLK: now also IC2.20 (B1), J13.1 (Pin_1)
- net LED_SPI_MOSI: now also IC2.18 (B2), J12.1 (Pin_1)
- net at D8.6 (DO): now also J14.1 (Pin_1)
- net at D8.5 (CO): now also J16.1 (Pin_1)
- net at L2.1: now also C2.1, U2.1 (SW), U2.2 (SW), U2.3 (SW)
- net at D12.1 (DI): now also J15.1 (Pin_1)
- net at D7.5 (CO): now also J11.1 (Pin_1)
- net at D7.6 (DO): now also J10.1 (Pin_1)
- net at R4.2: now also U2.6 (RT)
- net at C13.1, R2.1, R6.2: now also U2.7 (FB)
- net at R13.2: now also USB-C2.A5 (CC1)
- net at BUT2.1: now also R15.1
- net at R14.2: now also USB-C2.B5 (CC2)
- net at D12.2 (CI): now also J17.1 (Pin_1)
- net GPIO1: no longer names the net of U4.39 (IO1/RTC_GPIO1/GPIO1/TOUCH1/ADC1_CH0)
- net GPIO10\FSPICS0(SPI3_CS0): no longer names the net of U4.18 (IO10/RTC_GPIO10/GPIO10/TOUCH10/ADC1_CH9/FSPICS0/FSPIIO4/SUBSPICS0)
- net GPIO13\FSPIQ(SPI3_MISO): no longer names the net of U4.21 (IO13/RTC_GPIO13/GPIO13/TOUCH13/ADC2_CH2/FSPIQ/FSPIIO7/SUBSPIQ)
- net GPIO14: no longer names the net of U4.22 (IO14/RTC_GPIO14/GPIO14/TOUCH14/ADC2_CH3/FSPIWP/FSPIDQS/SUBSPIWP)
- net GPIO15: no longer names the net of U4.8 (IO15/RTC_GPIO15/GPIO15/U0RTS/ADC2_CH4/XTAL_32K_P)
- net GPIO16: no longer names the net of U4.9 (IO16/RTC_GPIO16/GPIO16/U0CTS/ADC2_CH5/XTAL_32K_N)
- net GPIO17\U1TXD: no longer names the net of U4.10 (IO17/RTC_GPIO17/GPIO17/U1TXD/ADC2_CH6)
- net GPIO18\U1RXD: no longer names the net of U4.11 (IO18/RTC_GPIO18/GPIO18/U1RXD/ADC2_CH7/CLK_OUT3)
- net GPIO2: no longer names the net of U4.38 (IO2/RTC_GPIO2/GPIO2/TOUCH2/ADC1_CH1)
- net GPIO21: no longer names the net of U4.23 (IO21/RTC_GPIO21/GPIO21)
- net GPIO3: no longer names the net of U4.15 (IO3/RTC_GPIO3/GPIO3/TOUCH3/ADC1_CH2)
- net GPIO3: now also R5.1
- net GPIO35: no longer names the net of U4.28 (IO35*/SPIIO6/GPIO35/FSPID/SUBSPID)
- net GPIO36: no longer names the net of U4.29 (IO36*/SPIIO7/GPIO36/FSPICLK/SUBSPICLK)
- net GPIO37: no longer names the net of U4.30 (IO37*/SPIDQS/GPIO37/FSPIQ/SUBSPIQ)
- net GPIO38\LED1: no longer names the net of U4.31 (IO38/GPIO38/FSPIWP/SUBSPIWP)
- net GPIO39: no longer names the net of U4.32 (IO39/MTCK/GPIO39/CLK_OUT3/SUBSPICS1)
- net GPIO4: no longer names the net of U4.4 (IO4/RTC_GPIO4/GPIO4/TOUCH4/ADC1_CH3)
- net GPIO40: no longer names the net of U4.33 (IO40/MTDO/GPIO40/CLK_OUT2)
- net GPIO41: no longer names the net of U4.34 (IO41/MTDI/GPIO41/CLK_OUT1)
- net GPIO42: no longer names the net of U4.35 (IO42/MTMS/GPIO42)
- net GPIO43\U0TXD: no longer names the net of U4.37 (TXD0/U0TXD/GPIO43/CLK_OUT1)
- net GPIO44\U0RXD: no longer names the net of U4.36 (RXD0/U0RXD/GPIO44/CLK_OUT2)
- net GPIO45: no longer names the net of U4.26 (IO45/GPIO45)
- net GPIO46: no longer names the net of U4.16 (IO46/GPIO46)
- net GPIO47\I2C_SCL: no longer names the net of U4.24 (IO47/SPICLK_P_DIFF/GPIO47/SUBSPICLK_P_DIFF)
- net GPIO48\I2C_SDA: no longer names the net of U4.25 (IO48/SPICLK_N_DIFF/GPIO48/SUBSPICLK_N_DIFF)
- net GPIO6\BAT_SENS: no longer names the net of U4.6 (IO6/RTC_GPIO6/GPIO6/TOUCH6/ADC1_CH5)
- net GPIO7: no longer names the net of U4.7 (IO7/RTC_GPIO7/GPIO7/TOUCH7/ADC1_CH6)
- net GPIO8: no longer names the net of U4.12 (IO8/RTC_GPIO8/GPIO8/TOUCH8/ADC1_CH7/SUBSPICS1)
- net GPIO9: no longer names the net of U4.17 (IO9/RTC_GPIO9/GPIO9/TOUCH9/ADC1_CH8/FSPIHD/SUBSPIHD)
- new net: C2.2, U2.4 (BOOT)
- new net: D2.2 (A), USB-C2.A4 (VBUS), USB-C2.A9 (VBUS), USB-C2.B4 (VBUS), USB-C2.B9 (VBUS)
- no-connect marks 15 -> 44
Other:
- note removed: "*NC"
- note removed: "USER LED"
- moved on the sheet: BUT2, C13, C14, C15, C19, C20, C21, RST2
