File: rover_bms_ble_controller_hw/rover_bms_ble_controller_hw.kicad_pcb (KiCad board)
At the start: 2 copper layers, 100 x 20 mm, 61 parts, among them T2 BC817-40(SOT23), T3 BC817-40(SOT23), U2 SY8089AAAC(SOT23-5), U3 ESP32-S3-WROOM-1-N8R8, U4 CH340X(MSOP-10)

Commit message: Update
Parts:
- removed the C2 at (145.1, 9.36)
- removed the C5 at (145.1, 14.9)
- removed the D4 at (178.0, 21.6)
- removed R19, R20: 5.1k/R0603, OLIMEX_RLC-FP:R_0603_5MIL_DWS
- removed R21: 100R/R0402, OLIMEX_RLC-FP:R_0402_5MIL_DWS
- removed R22, R23: 0k/R0603, OLIMEX_RLC-FP:R_0603_5MIL_DWS
- removed T2, T3: BC817-40(SOT23), OLIMEX_Transistors-FP:SOT23
- removed the U4 at (190.5, 11.0)
- removed USB-UART2: USB-C-16P-F(A40-00119-A52-12), OLIMEX_Connectors-FP:USB2.0_TYPE-C(A40-00119-A52-12)
- removed pUEXT2: BM10B-SRSS-TB, OLIMEX_Connectors-FP:BM10B-SRSS-TB
- added C10: 47uF/50V, Capacitor_SMD:CP_Elec_6.3x7.7, B.Cu at (157.5, 90.0)
- added C11: 47uF/6.3V, OLIMEX_RLC-FP:C_0603_5MIL_DWS, F.Cu at (144.7, 40.2)
- added C11: 100nF/50V, OLIMEX_RLC-FP:C_0603_5MIL_DWS, F.Cu at (1.40, 12.0)
- added C12: 33pF/50V, OLIMEX_RLC-FP:C_0603_5MIL_DWS, F.Cu at (1.40, 14.8)
- added C12: 100nF/10V, OLIMEX_RLC-FP:C_0402_5MIL_DWS, F.Cu at (152.8, 36.5)
- added C13: 33pF/10V, OLIMEX_RLC-FP:C_0402_5MIL_DWS, F.Cu at (152.8, 38.6)
- added C13: 22uF/6.3V/20%/X5R/C0603, OLIMEX_RLC-FP:C_0603_5MIL_DWS, F.Cu at (195.5, 53.5)
- added C14: 100nF/10V/10%/X7R/C0402, OLIMEX_RLC-FP:C_0402_5MIL_DWS, F.Cu at (195.5, 67.5)
- added C15: 22uF/6.3V/20%/X5R/C0603, OLIMEX_RLC-FP:C_0603_5MIL_DWS, B.Cu at (126.3, 64.5)
- added C16: 22uF/6.3V/20%/X5R/C0603, OLIMEX_RLC-FP:C_0603_5MIL_DWS, F.Cu at (195.5, 58.0)
- added C17: 1uF/10V/10%/X5R/C0603, OLIMEX_RLC-FP:C_0603_5MIL_DWS, F.Cu at (195.5, 62.5)
- added C18: 22uF/6.3V/20%/X5R/C0603, OLIMEX_RLC-FP:C_0603_5MIL_DWS, F.Cu at (131.0, 51.5)
- added C19: 100nF/10V/10%/X7R/C0402, OLIMEX_RLC-FP:C_0402_5MIL_DWS, B.Cu at (89.0, 92.0)
- added C2: 100nF/50V, OLIMEX_RLC-FP:C_0402_5MIL_DWS, F.Cu at (147.8, 34.3)
- added C2: 100uF/50V, Capacitor_SMD:CP_Elec_8x10.5, B.Cu at (141.5, 81.3)
- added C20: 100nF/10V/10%/X7R/C0402, OLIMEX_RLC-FP:C_0402_5MIL_DWS, B.Cu at (91.0, 86.0)
- added C21: 22uF/6.3V/20%/X5R/C0603, OLIMEX_RLC-FP:C_0603_5MIL_DWS, F.Cu at (131.6, 47.5)
- added C5: 4.7uF/50V, OLIMEX_RLC-FP:C_0402_5MIL_DWS, F.Cu at (147.8, 38.6)
- added C5: 100nF/50V, OLIMEX_RLC-FP:C_0603_5MIL_DWS, B.Cu at (132.5, 84.0)
- added C8: 1nF/50V, OLIMEX_RLC-FP:C_0603_5MIL_DWS, F.Cu at (1.40, 9.22)
- added C8: 100nF/10V, OLIMEX_RLC-FP:C_0402_5MIL_DWS, F.Cu at (150.3, 38.6)
- added C9: 1nF/10V, OLIMEX_RLC-FP:C_0402_5MIL_DWS, F.Cu at (152.8, 34.3)
- added C9: 47uF/50V, Capacitor_SMD:CP_Elec_6.3x7.7, B.Cu at (147.5, 90.0)
- added C_BOOT2: 100nF/50V, OLIMEX_RLC-FP:C_0603_5MIL_DWS, B.Cu at (129.0, 81.5)
- added IC2: TXS0108E, TXS0108E:PW_R-PDSO-G20, B.Cu at (86.5, 87.5)
- added L3: 2.2uH/1.5A/DCR=72mR/20%/3.00x3.00x1.50mm/CD32(NR3015T2R2M), OLIMEX_RLC-FP:CD32, B.Cu at (117.3, 62.0)
- added U3: SY8089AAAC(SOT23-5), OLIMEX_Regulators-FP:SOT-23-5, B.Cu at (122.3, 62.0)
- C3: value 100nF/10V/10%/X7R/C0402 -> 4.7uF/50V; footprint OLIMEX_RLC-FP:C_0402_5MIL_DWS -> Capacitor_SMD:CP_Elec_4x5.7; moved to B.Cu
- C4: value 22uF/6.3V/20%/X5R/C0603 -> 4.7uF/50V; footprint OLIMEX_RLC-FP:C_0603_5MIL_DWS -> Capacitor_SMD:CP_Elec_4x5.7; moved to B.Cu
- C6: value 100nF/10V/10%/X7R/C0402 -> 1nF/50V; footprint OLIMEX_RLC-FP:C_0402_5MIL_DWS -> OLIMEX_RLC-FP:C_0603_5MIL_DWS; moved to B.Cu
- C7: value 1uF/10V/10%/X5R/C0603 -> 100nF/50V
- D2, D3: moved to B.Cu
- L2: value 2.2uH/1.5A/DCR=72mR/20%/3.00x3.00x1.50mm/CD32(NR3015T2R2M) -> 4.7uH; footprint OLIMEX_RLC-FP:CD32 -> Inductor_SMD:L_Sunlord_MWSA1003S; moved to B.Cu
- R10: value 1k/R0402 -> 49.9k/1%/R0402; moved to B.Cu
- R11: value 5.1k/R0603 -> 10k/R0402; footprint OLIMEX_RLC-FP:R_0603_5MIL_DWS -> OLIMEX_RLC-FP:R_0402_5MIL_DWS
- R12: value 5.1k/R0603 -> 100k/R0603; moved to B.Cu
- R13: value 1k/R0402 -> 2.2k/R0402
- R14, R15: value 2.2k/R0402 -> 5.1k/R0603; footprint OLIMEX_RLC-FP:R_0402_5MIL_DWS -> OLIMEX_RLC-FP:R_0603_5MIL_DWS
- R16: value NA/R0402 -> 100R/R0402
- R17: value 2.2k/R0402 -> 0k/R0603; footprint OLIMEX_RLC-FP:R_0402_5MIL_DWS -> OLIMEX_RLC-FP:R_0603_5MIL_DWS
- R18: value 10k/R0402 -> 0k/R0603; footprint OLIMEX_RLC-FP:R_0402_5MIL_DWS -> OLIMEX_RLC-FP:R_0603_5MIL_DWS
- R2: value 220k/R0402 -> 10k/R0402
- R3: value 10k/R0402 -> 100k/R0603; footprint OLIMEX_RLC-FP:R_0402_5MIL_DWS -> OLIMEX_RLC-FP:R_0603_5MIL_DWS; moved to B.Cu
- R4: value 470k/R0402 -> 1k/R0603; footprint OLIMEX_RLC-FP:R_0402_5MIL_DWS -> OLIMEX_RLC-FP:R_0603_5MIL_DWS
- R5: value 220k/R0402 -> 31.6k/R0603; footprint OLIMEX_RLC-FP:R_0402_5MIL_DWS -> OLIMEX_RLC-FP:R_0603_5MIL_DWS; moved to B.Cu
- R6: value 49.9k/1%/R0402 -> 19.1k/R0603; footprint OLIMEX_RLC-FP:R_0402_5MIL_DWS -> OLIMEX_RLC-FP:R_0603_5MIL_DWS; moved to B.Cu
- R7: value 10k/R0402 -> 220k/R0402
- R8: value 100R/R0402 -> 220k/R0402; moved to B.Cu
- R9: value 4.7k/R0402 -> 470k/R0402
- U2: value SY8089AAAC(SOT23-5) -> LMR51450SDRRR; footprint OLIMEX_Regulators-FP:SOT-23-5 -> Libs:CONV_LMR51450SDRRR; moved to B.Cu
- moved C7 144.1 mm to (1.40, 6.45)
- moved LED2 112.1 mm to (87.5, 94.5), turned to 180 degrees
- moved R12 103.0 mm to (89.5, 93.5), turned to 180 degrees
- moved R13 102.4 mm to (84.5, 94.5)
- moved L2 95.6 mm to (130.5, 91.5)
- moved USB-OTG2 89.9 mm to (72.0, 118.0)
- moved C6 76.8 mm to (132.5, 85.5)
- moved R17 74.3 mm to (163.5, 89.5), turned to 90 degrees
- moved C3 73.5 mm to (155.0, 82.5), turned to -90 degrees
- moved R6 73.5 mm to (135.5, 80.0), turned to 90 degrees
- moved C4 70.5 mm to (150.0, 82.5), turned to -90 degrees
- moved U2 69.2 mm to (132.0, 81.0)
- moved D2 67.9 mm to (127.8, 61.0)
- moved BUT2 66.1 mm to (239.5, 52.0)
- moved R16 64.4 mm to (180.0, 73.5)
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- renumbered D11 to D10, D12 to D11, D13 to D12, D14 to D13, D5 to D4, D6 to D5, D7 to D6, D8 to D7, D9 to D8, D10 to D9, U3 to U4
Connections:
- C3 pad 1: GND -> +24V
- C3 pad 2: +3.3V -> GND
- C4 pad 1: Net-(D2-K) -> +24V
- C6 pad 1: +3.3V -> GND
- C6 pad 2: GND -> +24V
- C7 pad 1: /TOP/MCU&LEDS/ESP_EN -> GND
- C7 pad 2: GND -> +5V
- D13 pad 1: Net-(D14-DI) -> Net-(D13-DI)
- D13 pad 2: Net-(D14-CI) -> Net-(D13-CI)
- D4 pad 1: /TOP/MCU&LEDS/GPIO11\FSPID(SPI3_MOSI) -> /TOP/MCU&LEDS/LED_SPI_MOSI
- D4 pad 2: /TOP/MCU&LEDS/GPIO12\FSPICLK(SPI3_CLK) -> /TOP/MCU&LEDS/LED_SPI_CLK
- D8 pad 5: Net-(D9-CO) (its old number) -> Net-(D8-CO)
- D8 pad 6: Net-(D9-DO) (its old number) -> Net-(D8-DO)
- L2 pad 1: Net-(U2-LX) -> Net-(C_BOOT2-~-Pad1)
- L2 pad 2: +3.3V -> +5V
- LED_DI/CI2 pad 1: /TOP/MCU&LEDS/GPIO11\FSPID(SPI3_MOSI) -> /TOP/MCU&LEDS/LED_SPI_MOSI
- LED_DI/CI2 pad 2: /TOP/MCU&LEDS/GPIO12\FSPICLK(SPI3_CLK) -> /TOP/MCU&LEDS/LED_SPI_CLK
- LED_DI/CI3 pad 1: Net-(D14-DI) -> Net-(D13-DI)
- LED_DI/CI3 pad 2: Net-(D14-CI) -> Net-(D13-CI)
- LED_DO/CO2 pad 1: Net-(D9-DO) (its old number) -> Net-(D8-DO)
- LED_DO/CO2 pad 2: Net-(D9-CO) (its old number) -> Net-(D8-CO)
- R10 pad 1: Net-(T3-E) -> Net-(U3-FB)
- R10 pad 2: Net-(T2-B) -> GND
- R11 pad 1: GND -> +3.3V
- R11 pad 2: Net-(USB-UART2-CC2) -> /TOP/MCU&LEDS/ESP_EN
- R12 pad 2: Net-(USB-UART2-CC1) -> +3.3V
- R13 pad 1: Net-(T2-E) -> +3.3V
- R13 pad 2: Net-(T3-B) -> Net-(LED2-A)
- R14 pad 1: +3.3V -> GND
- R14 pad 2: /TOP/MCU&LEDS/GPIO47\I2C_SCL -> Net-(USB-OTG2-CC1)
- R15 pad 1: +3.3V -> GND
- R15 pad 2: Net-(LED2-A) -> Net-(USB-OTG2-CC2)
- R16 pad 1: +3.3V -> /TOP/MCU&LEDS/GPIO0\BUT1
- R16 pad 2: /TOP/MCU&LEDS/GPIO0\BUT1 -> Net-(BUT2-~-Pad1)
- R17 pad 1: +3.3V -> Net-(D13-DI)
- R17 pad 2: /TOP/MCU&LEDS/GPIO48\I2C_SDA -> Net-(D8-CO)
- R18 pad 1: +3.3V -> Net-(D13-CI)
- R18 pad 2: /TOP/MCU&LEDS/GPIO10\FSPICS0(SPI3_CS0) -> Net-(D8-DO)
- R2 pad 1: +5V -> +3.3V
- R2 pad 2: /TOP/MCU&LEDS/GPIO5\PWR_SENS -> /TOP/MCU&LEDS/GPIO3
- R3 pad 1: +3.3V -> Net-(U2-FB)
- R3 pad 2: /TOP/MCU&LEDS/GPIO3 -> +5V
- R4 pad 1: /TOP/MCU&LEDS/GPIO5\PWR_SENS -> Net-(C12-~-Pad2)
- R4 pad 2: GND -> +5V
- R5 pad 1: Net-(U2-FB) -> GND
- R5 pad 2: +3.3V -> Net-(U2-RT)
- R6 pad 1: Net-(U2-FB) -> GND
- R6 pad 2: GND -> Net-(U2-FB)
- R7 pad 1: +3.3V -> +5V
- R7 pad 2: /TOP/MCU&LEDS/ESP_EN -> /TOP/MCU&LEDS/GPIO5\PWR_SENS
- R8 pad 1: Net-(U4-TXD) -> Net-(U3-FB)
- R8 pad 2: /TOP/MCU&LEDS/GPIO44\U0RXD -> +3.3V
- R9 pad 1: Net-(U4-CTS#) -> /TOP/MCU&LEDS/GPIO5\PWR_SENS
- R9 pad 2: Net-(T3-E) -> GND
- U2 pad 1: Net-(D2-K) -> Net-(C_BOOT2-~-Pad1)
- U2 pad 2: GND -> Net-(C_BOOT2-~-Pad1)
- U2 pad 3: Net-(U2-LX) -> Net-(C_BOOT2-~-Pad1)
- U2 pad 4: Net-(D2-K) -> Net-(U2-BOOT)
- U2 pad 5: Net-(U2-FB) -> unconnected-(U2-PG-Pad5)
- USB-OTG2 pad A4: Net-(D4-A) -> Net-(D3-A)
- USB-OTG2 pad A9: Net-(D4-A) -> Net-(D3-A)
- USB-OTG2 pad B4: Net-(D4-A) -> Net-(D3-A)
- USB-OTG2 pad B9: Net-(D4-A) -> Net-(D3-A)
Routing:
- net /TOP/MCU&LEDS/LED_SPI_MOSI: track 0.00 -> 25.9 mm
- net /TOP/MCU&LEDS/LED_SPI_CLK: track 0.00 -> 23.6 mm
- net +3.3V: track 0.00 -> 21.3 mm, vias 0 -> 1
- net +5V: track 110.1 -> 127.8 mm, vias 0 -> 2
- net Net-(D13-CI): track 0.00 -> 16.6 mm
- net Net-(D8-CO): track 0.00 -> 15.0 mm
- net Net-(D2-K): track 0.00 -> 9.07 mm
- net Net-(D13-DI): track 0.00 -> 8.69 mm
- net GND: track 0.00 -> 8.30 mm
- net Net-(D8-DO): track 0.00 -> 7.19 mm
- net Net-(D14-CI): track 7.01 -> 0.00 mm
- net Net-(D14-DI): track 6.88 -> 0.00 mm
- net Net-(D9-CO) (its old number): track 6.82 -> 0.00 mm
- net Net-(D9-CO): track 0.00 -> 6.80 mm
- net +24V: track 0.00 -> 6.71 mm
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- added copper zone on B.Cu, net +24V
- added copper zone on B.Cu, net +5V
- added copper zone on B.Cu, net Net-(C_BOOT2-~-Pad1)
Other:
- board size 100 x 20 mm -> 100 x 24 mm

Commit message: Final version
Parts:
- removed the C11 at (144.7, 40.2)
- removed the C11 at (1.40, 12.0)
- removed the C13 at (152.8, 38.6)
- removed the C16 at (195.5, 58.0)
- removed the C19 at (89.0, 92.0)
- removed the C5 at (147.8, 38.6)
- removed the C7 at (1.40, 6.45)
- removed the C8 at (1.40, 9.22)
- removed the C8 at (150.3, 38.6)
- removed C_BOOT2: 100nF/50V, OLIMEX_RLC-FP:C_0603_5MIL_DWS
- removed the D3 at (132.0, 63.0)
- removed LED2: LED/Green/0603, OLIMEX_LEDs-FP:LED_0603_KA
- removed LED_DI/CI2, LED_DI/CI3, LED_DO/CO2, LED_DO/CO3: DW02S, OLIMEX_Connectors-FP:LIPO_BAT_VERTICAL_DW02S
- removed the R13 at (84.5, 94.5)
- removed R16: 100R/R0402, OLIMEX_RLC-FP:R_0402_5MIL_DWS
- removed R17, R18: 0k/R0603, OLIMEX_RLC-FP:R_0603_5MIL_DWS
- removed the R2 at (178.5, 57.5)
- removed USB-OTG2: USB-C-16P-F(A40-00119-A52-12), OLIMEX_Connectors-FP:USB2.0_TYPE-C(A40-00119-A52-12)
- added C17: 47uF/50V, Capacitor_SMD:CP_Elec_6.3x7.7, B.Cu at (111.0, 80.5)
- added C22: 100nF/50V/0603, Capacitor_SMD:C_0603_1608Metric, B.Cu at (78.2, 87.2)
- added C8: 100nF/50V/0603, Capacitor_SMD:C_0603_1608Metric, B.Cu at (140.5, 89.5)
- added J10: DO_OUT, MechatronicsAcademy:TestPoint_Pad, F.Cu at (165.5, 78.0)
- added J11: CO_OUT, MechatronicsAcademy:TestPoint_Pad, F.Cu at (165.5, 80.0)
- added J12: DO_IN, MechatronicsAcademy:TestPoint_Pad, F.Cu at (69.5, 78.0)
- added J13: CI_IN, MechatronicsAcademy:TestPoint_Pad, F.Cu at (69.5, 80.0)
- added J14: DO_OUT_2, MechatronicsAcademy:TestPoint_Pad, F.Cu at (69.5, 91.0)
- added J15: DI_IN_2, MechatronicsAcademy:TestPoint_Pad, F.Cu at (165.5, 91.0)
- added J16: CO_OUT_2, MechatronicsAcademy:TestPoint_Pad, F.Cu at (69.5, 93.0)
- added J17: CI_IN_2, MechatronicsAcademy:TestPoint_Pad, F.Cu at (165.5, 93.0)
- added J2: +24V_PAD, MechatronicsAcademy:TestPoint_Pad_1, B.Cu at (159.2, 79.2)
- added J3: IN_+5, MechatronicsAcademy:TestPoint_Pad_1, F.Cu at (70.2, 85.5)
- added J4: OUT_+5, MechatronicsAcademy:TestPoint_Pad_1, F.Cu at (164.8, 85.5)
- added J5: GND_IN, MechatronicsAcademy:TestPoint_Pad_1, F.Cu at (164.8, 95.8)
- added J6: GND_OUT, MechatronicsAcademy:TestPoint_Pad_1, F.Cu at (70.2, 75.2)
- added J7: GND_PAD, MechatronicsAcademy:TestPoint_Pad_1, B.Cu at (164.5, 79.5)
- added J8: GND_IN, MechatronicsAcademy:TestPoint_Pad_1, F.Cu at (164.8, 75.2)
- added J9: GND_OUT, MechatronicsAcademy:TestPoint_Pad_1, F.Cu at (70.2, 95.8)
- added R15: 100/R0603, Resistor_SMD:R_0603_1608Metric_Pad0.98x0.95mm_HandSolder, B.Cu at (75.0, 89.5)
- added R5: 10k/R0603, Resistor_SMD:R_0603_1608Metric_Pad0.98x0.95mm_HandSolder, B.Cu at (101.5, 94.0)
- added USB-C2: USB2.0_TYPE-C(A40-00119-A52-12), MechatronicsAcademy:USB2.0_TYPE-C-ONLY-PADS, B.Cu at (109.5, 98.2)
- BUT2, RST2: moved to B.Cu
- C12: value 100nF/10V -> 100nF/50V/0603; footprint OLIMEX_RLC-FP:C_0402_5MIL_DWS -> Capacitor_SMD:C_0603_1608Metric; moved to B.Cu
- C13: renamed from C12; value 33pF/50V -> 33pF/50V/0603; footprint OLIMEX_RLC-FP:C_0603_5MIL_DWS -> Capacitor_SMD:C_0603_1608Metric; moved to B.Cu
- C14: renamed from C13; value 22uF/6.3V/20%/X5R/C0603 -> 22uF/10V/X5R/0603; footprint OLIMEX_RLC-FP:C_0603_5MIL_DWS -> Capacitor_SMD:C_0603_1608Metric; moved to B.Cu
- C15: renamed from C14; value 100nF/10V/10%/X7R/C0402 -> 100nF/50V/0603; footprint OLIMEX_RLC-FP:C_0402_5MIL_DWS -> Capacitor_SMD:C_0603_1608Metric; moved to B.Cu
- C16: renamed from C15; value 22uF/6.3V/20%/X5R/C0603 -> 22uF/10V/X5R/0603; footprint OLIMEX_RLC-FP:C_0603_5MIL_DWS -> Capacitor_SMD:C_0603_1608Metric
- C18: renamed from C17; value 1uF/10V/10%/X5R/C0603 -> 1uF/10V/X5R/0603; footprint OLIMEX_RLC-FP:C_0603_5MIL_DWS -> Capacitor_SMD:C_0603_1608Metric; moved to B.Cu
- C19: renamed from C20; value 100nF/10V/10%/X7R/C0402 -> 100nF/50V/0603; footprint OLIMEX_RLC-FP:C_0402_5MIL_DWS -> Capacitor_SMD:C_0603_1608Metric
- C2: value 100nF/50V -> 100nF/50V/0603; footprint OLIMEX_RLC-FP:C_0402_5MIL_DWS -> Capacitor_SMD:C_0603_1608Metric; moved to B.Cu
- C20: renamed from C21; value 22uF/6.3V/20%/X5R/C0603 -> 22uF/10V/X5R/0603; footprint OLIMEX_RLC-FP:C_0603_5MIL_DWS -> Capacitor_SMD:C_0603_1608Metric; moved to B.Cu
- C21: renamed from C18; value 22uF/6.3V/20%/X5R/C0603 -> 22uF/10V/X5R/0603; footprint OLIMEX_RLC-FP:C_0603_5MIL_DWS -> Capacitor_SMD:C_0603_1608Metric; moved to B.Cu
- C6: renamed from C5; value 100nF/50V -> 100nF/50V/0603; footprint OLIMEX_RLC-FP:C_0603_5MIL_DWS -> Capacitor_SMD:C_0603_1608Metric
- C7: renamed from C6; value 1nF/50V -> 1nF/50V/0603; footprint OLIMEX_RLC-FP:C_0603_5MIL_DWS -> Capacitor_SMD:C_0603_1608Metric
- C9: value 1nF/10V -> 1nF/50V/0603; footprint OLIMEX_RLC-FP:C_0402_5MIL_DWS -> Capacitor_SMD:C_0603_1608Metric; moved to B.Cu
- D10: renamed from D11; value APA102 -> SK9822
- D11: renamed from D12; value APA102 -> SK9822
- D12: renamed from D13; value APA102 -> SK9822
- D3: renamed from D4; value APA102 -> SK9822
- D4: renamed from D5; value APA102 -> SK9822
- D5: renamed from D6; value APA102 -> SK9822
- D6: renamed from D7; value APA102 -> SK9822
- D7: renamed from D8; value APA102 -> SK9822
- D8: renamed from D9; value APA102 -> SK9822
- D9: renamed from D10; value APA102 -> SK9822
- IC2: footprint TXS0108E:PW_R-PDSO-G20 -> MechatronicsAcademy:PW_R-PDSO-G20
- R10: value 49.9k/1%/R0402 -> 49.9k/1%/R0603; footprint OLIMEX_RLC-FP:R_0402_5MIL_DWS -> Resistor_SMD:R_0603_1608Metric_Pad0.98x0.95mm_HandSolder
- R11: value 10k/R0402 -> 10k/R0603; footprint OLIMEX_RLC-FP:R_0402_5MIL_DWS -> Resistor_SMD:R_0603_1608Metric_Pad0.98x0.95mm_HandSolder; moved to B.Cu
- R12, R6: footprint OLIMEX_RLC-FP:R_0603_5MIL_DWS -> Resistor_SMD:R_0603_1608Metric_Pad0.98x0.95mm_HandSolder
- R13: renamed from R14; footprint OLIMEX_RLC-FP:R_0603_5MIL_DWS -> Resistor_SMD:R_0603_1608Metric_Pad0.98x0.95mm_HandSolder; moved to B.Cu
- R14: renamed from R15; footprint OLIMEX_RLC-FP:R_0603_5MIL_DWS -> Resistor_SMD:R_0603_1608Metric_Pad0.98x0.95mm_HandSolder; moved to B.Cu
- R2: renamed from R3; footprint OLIMEX_RLC-FP:R_0603_5MIL_DWS -> Resistor_SMD:R_0603_1608Metric_Pad0.98x0.95mm_HandSolder
- R3: renamed from R4; footprint OLIMEX_RLC-FP:R_0603_5MIL_DWS -> Resistor_SMD:R_0603_1608Metric_Pad0.98x0.95mm_HandSolder; moved to B.Cu
- R4: renamed from R5; footprint OLIMEX_RLC-FP:R_0603_5MIL_DWS -> Resistor_SMD:R_0603_1608Metric_Pad0.98x0.95mm_HandSolder
- R7: value 220k/R0402 -> 2200k/R0603; footprint OLIMEX_RLC-FP:R_0402_5MIL_DWS -> Resistor_SMD:R_0603_1608Metric_Pad0.98x0.95mm_HandSolder; moved to B.Cu
- R8: value 220k/R0402 -> 220k/R0603; footprint OLIMEX_RLC-FP:R_0402_5MIL_DWS -> Resistor_SMD:R_0603_1608Metric_Pad0.98x0.95mm_HandSolder
- R9: value 470k/R0402 -> 470k/R0603; footprint OLIMEX_RLC-FP:R_0402_5MIL_DWS -> Resistor_SMD:R_0603_1608Metric_Pad0.98x0.95mm_HandSolder; moved to B.Cu
- U2: footprint Libs:CONV_LMR51450SDRRR -> MechatronicsAcademy:LMR51450SDRRR
- moved BUT2 173.2 mm to (70.8, 91.5), turned to 90 degrees
- moved RST2 164.7 mm to (70.8, 85.0), turned to -90 degrees
- moved C13 145.8 mm to (133.0, 77.5), turned to 180 degrees
- moved C14 93.1 mm to (105.0, 75.5), turned to 90 degrees
- moved C18 92.9 mm to (104.0, 79.0)
- moved R14 91.2 mm to (106.0, 91.5), turned to -90 degrees
- moved C15 88.8 mm to (107.0, 75.5), turned to -90 degrees
- moved R13 84.9 mm to (110.0, 91.0), turned to -90 degrees
- moved R9 80.2 mm to (103.5, 81.5), turned to 180 degrees
- moved R7 78.3 mm to (103.5, 83.5)
- moved R11 76.3 mm to (103.0, 76.5), turned to -90 degrees
- moved C21 64.6 mm to (78.2, 88.8), turned to 180 degrees
- moved C20 59.7 mm to (80.0, 77.5)
- moved C9 56.1 mm to (142.5, 89.5), turned to -90 degrees
- moved C12 53.8 mm to (162.0, 89.5), turned to -90 degrees
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- renumbered C9 to C10, C10 to C11, C2 to C3, C3 to C4, C4 to C5
Connections:
- C12 pad 1: +5V -> GND
- C12 pad 2: GND -> +5V
- C16 pad 1: Net-(D2-K) -> +5V
- C9 pad 1: +5V -> GND
- C9 pad 2: GND -> +5V
- D2 pad 1: Net-(D2-K) -> +5V
- D2 pad 2: +5V -> Net-(D2-A)
- IC2 pad 1: /TOP/MCU&LEDS/GPIO11\FSPID(SPI3_MOSI) -> /TOP/MCU&LEDS/GPIO12\FSPICLK(SPI3_CLK)
- IC2 pad 18: /TOP/MCU&LEDS/LED_SPI_CLK -> /TOP/MCU&LEDS/LED_SPI_MOSI
- IC2 pad 20: /TOP/MCU&LEDS/LED_SPI_MOSI -> /TOP/MCU&LEDS/LED_SPI_CLK
- IC2 pad 3: /TOP/MCU&LEDS/GPIO12\FSPICLK(SPI3_CLK) -> /TOP/MCU&LEDS/GPIO11\FSPID(SPI3_MOSI)
- L2 pad 1: Net-(C_BOOT2-~-Pad1) -> Net-(C2-~-Pad1)
- R7 pad 1: +5V -> /TOP/MCU&LEDS/GPIO5\PWR_SENS
- R7 pad 2: /TOP/MCU&LEDS/GPIO5\PWR_SENS -> +5V
- R9 pad 1: /TOP/MCU&LEDS/GPIO5\PWR_SENS -> GND
- R9 pad 2: GND -> /TOP/MCU&LEDS/GPIO5\PWR_SENS
- U2 pad 1: Net-(C_BOOT2-~-Pad1) -> Net-(C2-~-Pad1)
- U2 pad 2: Net-(C_BOOT2-~-Pad1) -> Net-(C2-~-Pad1)
- U2 pad 3: Net-(C_BOOT2-~-Pad1) -> Net-(C2-~-Pad1)
- U3 pad 1: Net-(D2-K) -> +5V
- U3 pad 4: Net-(D2-K) -> +5V
- U4 pad 10: /TOP/MCU&LEDS/GPIO17\U1TXD -> unconnected-(U4-IO17/RTC_GPIO17/GPIO17/U1TXD/ADC2_CH6-Pad10)
- U4 pad 11: /TOP/MCU&LEDS/GPIO18\U1RXD -> unconnected-(U4-IO18/RTC_GPIO18/GPIO18/U1RXD/ADC2_CH7/CLK_OUT3-Pad11)
- U4 pad 12: /TOP/MCU&LEDS/GPIO8 -> unconnected-(U4-IO8/RTC_GPIO8/GPIO8/TOUCH8/ADC1_CH7/SUBSPICS1-Pad12)
- U4 pad 15: /TOP/MCU&LEDS/GPIO3 -> Net-(U4-IO3/RTC_GPIO3/GPIO3/TOUCH3/ADC1_CH2)
- U4 pad 16: /TOP/MCU&LEDS/GPIO46 -> unconnected-(U4-IO46/GPIO46-Pad16)
- U4 pad 17: /TOP/MCU&LEDS/GPIO9 -> unconnected-(U4-IO9/RTC_GPIO9/GPIO9/TOUCH9/ADC1_CH8/FSPIHD/SUBSPIHD-Pad17)
- U4 pad 18: /TOP/MCU&LEDS/GPIO10\FSPICS0(SPI3_CS0) -> unconnected-(U4-IO10/RTC_GPIO10/GPIO10/TOUCH10/ADC1_CH9/FSPICS0/FSPIIO4/SUBSPICS0-Pad18)
- U4 pad 21: /TOP/MCU&LEDS/GPIO13\FSPIQ(SPI3_MISO) -> unconnected-(U4-IO13/RTC_GPIO13/GPIO13/TOUCH13/ADC2_CH2/FSPIQ/FSPIIO7/SUBSPIQ-Pad21)
- U4 pad 22: /TOP/MCU&LEDS/GPIO14 -> unconnected-(U4-IO14/RTC_GPIO14/GPIO14/TOUCH14/ADC2_CH3/FSPIWP/FSPIDQS/SUBSPIWP-Pad22)
- U4 pad 23: /TOP/MCU&LEDS/GPIO21 -> unconnected-(U4-IO21/RTC_GPIO21/GPIO21-Pad23)
- U4 pad 24: /TOP/MCU&LEDS/GPIO47\I2C_SCL -> unconnected-(U4-IO47/SPICLK_P_DIFF/GPIO47/SUBSPICLK_P_DIFF-Pad24)
- U4 pad 25: /TOP/MCU&LEDS/GPIO48\I2C_SDA -> unconnected-(U4-IO48/SPICLK_N_DIFF/GPIO48/SUBSPICLK_N_DIFF-Pad25)
- U4 pad 26: /TOP/MCU&LEDS/GPIO45 -> unconnected-(U4-IO45/GPIO45-Pad26)
- U4 pad 28: /TOP/MCU&LEDS/GPIO35 -> unconnected-(U4-IO35*/SPIIO6/GPIO35/FSPID/SUBSPID-Pad28)
- U4 pad 29: /TOP/MCU&LEDS/GPIO36 -> unconnected-(U4-IO36*/SPIIO7/GPIO36/FSPICLK/SUBSPICLK-Pad29)
- U4 pad 30: /TOP/MCU&LEDS/GPIO37 -> unconnected-(U4-IO37*/SPIDQS/GPIO37/FSPIQ/SUBSPIQ-Pad30)
- U4 pad 31: /TOP/MCU&LEDS/GPIO38\LED1 -> unconnected-(U4-IO38/GPIO38/FSPIWP/SUBSPIWP-Pad31)
- U4 pad 32: /TOP/MCU&LEDS/GPIO39 -> unconnected-(U4-IO39/MTCK/GPIO39/CLK_OUT3/SUBSPICS1-Pad32)
- U4 pad 33: /TOP/MCU&LEDS/GPIO40 -> unconnected-(U4-IO40/MTDO/GPIO40/CLK_OUT2-Pad33)
- U4 pad 34: /TOP/MCU&LEDS/GPIO41 -> unconnected-(U4-IO41/MTDI/GPIO41/CLK_OUT1-Pad34)
- U4 pad 35: /TOP/MCU&LEDS/GPIO42 -> unconnected-(U4-IO42/MTMS/GPIO42-Pad35)
- U4 pad 36: /TOP/MCU&LEDS/GPIO44\U0RXD -> unconnected-(U4-RXD0/U0RXD/GPIO44/CLK_OUT2-Pad36)
- U4 pad 37: /TOP/MCU&LEDS/GPIO43\U0TXD -> unconnected-(U4-TXD0/U0TXD/GPIO43/CLK_OUT1-Pad37)
- U4 pad 38: /TOP/MCU&LEDS/GPIO2 -> unconnected-(U4-IO2/RTC_GPIO2/GPIO2/TOUCH2/ADC1_CH1-Pad38)
- U4 pad 39: /TOP/MCU&LEDS/GPIO1 -> unconnected-(U4-IO1/RTC_GPIO1/GPIO1/TOUCH1/ADC1_CH0-Pad39)
- U4 pad 4: /TOP/MCU&LEDS/GPIO4 -> unconnected-(U4-IO4/RTC_GPIO4/GPIO4/TOUCH4/ADC1_CH3-Pad4)
- U4 pad 6: /TOP/MCU&LEDS/GPIO6\BAT_SENS -> unconnected-(U4-IO6/RTC_GPIO6/GPIO6/TOUCH6/ADC1_CH5-Pad6)
- U4 pad 7: /TOP/MCU&LEDS/GPIO7 -> unconnected-(U4-IO7/RTC_GPIO7/GPIO7/TOUCH7/ADC1_CH6-Pad7)
- U4 pad 8: /TOP/MCU&LEDS/GPIO15 -> unconnected-(U4-IO15/RTC_GPIO15/GPIO15/U0RTS/ADC2_CH4/XTAL_32K_P-Pad8)
- U4 pad 9: /TOP/MCU&LEDS/GPIO16 -> unconnected-(U4-IO16/RTC_GPIO16/GPIO16/U0CTS/ADC2_CH5/XTAL_32K_N-Pad9)
Routing:
- net +5V: track 127.8 -> 43.1 mm, vias 2 -> 7
- net +3.3V: track 21.3 -> 81.2 mm, vias 1 -> 0
- net /TOP/MCU&LEDS/ESP_EN: track 0.00 -> 42.5 mm, vias 0 -> 2
- net /TOP/MCU&LEDS/GPIO11\FSPID(SPI3_MOSI): track 6.68 -> 25.4 mm
- net /TOP/MCU&LEDS/GPIO19\USB_D-: track 0.00 -> 15.1 mm, vias 0 -> 2
- net /TOP/MCU&LEDS/GPIO12\FSPICLK(SPI3_CLK): track 8.91 -> 22.5 mm
- net /TOP/MCU&LEDS/GPIO20\USB_D+: track 0.00 -> 13.2 mm, vias 0 -> 2
- net /TOP/MCU&LEDS/LED_SPI_MOSI: track 25.9 -> 12.8 mm, vias 0 -> 1
- net /TOP/MCU&LEDS/GPIO0\BUT1: track 0.00 -> 12.6 mm, vias 0 -> 2
- net /TOP/MCU&LEDS/LED_SPI_CLK: track 23.6 -> 13.0 mm, vias 0 -> 1
- net Net-(D2-A): track 0.00 -> 9.88 mm
- net Net-(D7-CO): track 15.0 -> 5.85 mm
- net Net-(D2-K): track 9.07 -> 0.00 mm
- net GND: track 8.30 -> 16.4 mm, vias 0 -> 80
- net +24V: track 6.71 -> 0.50 mm
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- added copper zone on B.Cu, net +3.3V
- added copper zone on F.Cu, net +5V
- added copper zone on B.Cu, net Net-(C2-~-Pad1)
- added copper zone on B.Cu, net Net-(U3-FB)
- removed copper zone on B.Cu, net Net-(C_BOOT2-~-Pad1)
Other:
- board size 100 x 24 mm -> 100 x 25 mm
